File: pocket-to-dmg-ribbon/pocket-to-dmg-ribbon.kicad_pcb (KiCad board)
At the start: 2 copper layers, 34 x 28.4 mm, 2 parts, among them J1 DMG Ribbon, J2 MGB FPC

Commit message: Migrated some files to KiCad 7
Other:
- net class Default removed
